Commit message: Add files via upload

File: src/integ_description/urdf/arm.urdf.xacro (robot description, xacro)
@@ -10,8 +10,7 @@
   <xacro:property name="joint_radius" value="0.036"/>
   <xacro:property name="joint_length" value="0.05"/>
-  <xacro:property name="leg_length" value="0.80"/>
+  <xacro:property name="leg_length" value="0.00"/>
   <xacro:property name="arm_length" value="0.60"/>
-  <xacro:property name="hand_length" value="0.08"/>
-  <xacro:property name="finger_length" value="0.06"/>
+  <xacro:property name="hand_length" value="0.2"/>
   <!-- Materials -->
   <material name="orange">
@@ -39,7 +38,7 @@
       <xacro:insert_block name="origin"/>
       <mass value="${mass}"/>
-      <inertia ixx="${(mass/12)*(side*side+length*length)}"
+      <inertia ixx="${(mass/6)*(side*side)}"
                iyy="${(mass/12)*(side*side+length*length)}"
-               izz="${(mass/6)*(side*side)}"
+               izz="${(mass/12)*(side*side+length*length)}"
                ixy="0" ixz="0" iyz="0"/>
     </inertial>
@@ -110,13 +109,12 @@
   <!-- Joints Chain -->
   <xacro:arm_joint parent="leg" child="arm" axis="1 0 0" dist="${leg_length}"/>
-  <xacro:arm_joint parent="arm" child="hand" axis="0 0 1" dist="${arm_length}"/>
-  <xacro:arm_joint parent="hand" child="finger" axis="1 0 0" dist="${hand_length}"/>
+  <xacro:arm_joint parent="arm" child="hand" axis="1 0 0" dist="${arm_length}"/>
   <!-- End effector -->
-  <link name="finger">
-    <xacro:prism_vci length="${finger_length}" side="${link_side}">
-      <origin xyz="0 0 ${finger_length/2}" rpy="0 0 0"/>
+  <link name="hand">
+    <xacro:prism_vci length="${hand_length}" side="${link_side}">
+      <origin xyz="0 0 ${hand_length/2}" rpy="0 0 0"/>
     </xacro:prism_vci>
   </link>
-  <gazebo reference="finger">
+  <gazebo reference="hand">
     <material>Gazebo/Red</material>
   </gazebo>

Commit message: Update arm.urdf.xacro

File: src/integ_description/urdf/arm.urdf.xacro (robot description, xacro)
@@ -14,8 +14,8 @@
   <xacro:property name="hand_length" value="0.2"/>
   <!-- Materials -->
-  <material name="orange">
-    <color rgba="0.5 0.02 0.3 1.00"/>
+  <material name="noir">
+    <color rgba="0.1 0.1 0.1 1.00"/>
   </material>
-  <material name="gray">
+  <material name="blanc">
     <color rgba="0.80 0.80 0.80 1.00"/>
   </material>
@@ -30,5 +30,5 @@
     <visual>
       <xacro:prism_geometry/>
-      <material name="orange"/>
+      <material name="noir"/>
     </visual>
     <collision>
@@ -54,5 +54,5 @@
     <visual>
       <xacro:cylinder_geometry/>
-      <material name="gray"/>
+      <material name="blanc"/>
     </visual>
     <collision>
@@ -97,5 +97,5 @@
     </link>
     <gazebo reference="${parent}">
-      <material>Gazebo/Orange</material>
+      <material>Gazebo/noir</material>
     </gazebo>
   </xacro:macro>

Commit message: Suppressing collisions

File: src/integ_description/urdf/arm.urdf.xacro (robot description, xacro)
@@ -32,7 +32,4 @@
       <material name="noir"/>
     </visual>
-    <collision>
-      <xacro:prism_geometry/>
-    </collision>
     <inertial>
       <xacro:insert_block name="origin"/>
@@ -56,7 +53,4 @@
       <material name="blanc"/>
     </visual>
-    <collision>
-      <xacro:cylinder_geometry/>
-    </collision>
   </xacro:macro>
   <!-- Generates child joint of parent -->

Commit message: Robot gazebo

File: src/integ_description/urdf/arm.urdf.xacro (robot description, xacro)
@@ -10,16 +10,17 @@
   <xacro:property name="joint_radius" value="0.036"/>
   <xacro:property name="joint_length" value="0.05"/>
-  <xacro:property name="leg_length" value="0.00"/>
-  <xacro:property name="arm_length" value="0.60"/>
-  <xacro:property name="hand_length" value="0.2"/>
+  <xacro:property name="leg_length" value="0"/>
+  <xacro:property name="arm_length" value="0"/>
+  <xacro:property name="hand_length" value="0.8"/>
+  <xacro:property name="finger_length" value="0.6"/>
   <!-- Materials -->
-  <material name="noir">
-    <color rgba="0.1 0.1 0.1 1.00"/>
+  <material name="orange">
+    <color rgba="1.00 0.67 0.02 1.00"/>
   </material>
-  <material name="blanc">
+  <material name="gray">
     <color rgba="0.80 0.80 0.80 1.00"/>
   </material>
   <!-- Generates a box visual/collision/inertial -->
-  <xacro:macro name="prism_vci" params="side length mass:=1 *origin">
+  <xacro:macro name="prism_vci" params="side length mass:=0.1 *origin">
     <xacro:macro name="prism_geometry">
       <xacro:insert_block name="origin"/>
@@ -30,12 +31,12 @@
     <visual>
       <xacro:prism_geometry/>
-      <material name="noir"/>
+      <material name="orange"/>
     </visual>
     <inertial>
       <xacro:insert_block name="origin"/>
       <mass value="${mass}"/>
-      <inertia ixx="${(mass/6)*(side*side)}"
+      <inertia ixx="${(mass/12)*(side*side+length*length)}"
                iyy="${(mass/12)*(side*side+length*length)}"
-               izz="${(mass/12)*(side*side+length*length)}"
+               izz="${(mass/6)*(side*side)}"
                ixy="0" ixz="0" iyz="0"/>
     </inertial>
@@ -51,5 +52,5 @@
     <visual>
       <xacro:cylinder_geometry/>
-      <material name="blanc"/>
+      <material name="gray"/>
     </visual>
   </xacro:macro>
@@ -91,5 +92,5 @@
     </link>
     <gazebo reference="${parent}">
-      <material>Gazebo/noir</material>
+      <material>Gazebo/Orange</material>
     </gazebo>
   </xacro:macro>
@@ -99,16 +100,18 @@
   <joint name="world_foot_joint" type="fixed">
     <parent link="world"/>
-    <child link="leg"/>
+    <child link="arm"/>
   </joint>
+  <!--<xacro:arm_joint parent="world" child="arm" axis="0 0 1" dist="0"/>-->
   <!-- Joints Chain -->
-  <xacro:arm_joint parent="leg" child="arm" axis="1 0 0" dist="${leg_length}"/>
+  <!--<xacro:arm_joint parent="leg" child="arm" axis="0 0 1" dist="${leg_length}"/>-->
   <xacro:arm_joint parent="arm" child="hand" axis="1 0 0" dist="${arm_length}"/>
+  <xacro:arm_joint parent="hand" child="finger" axis="1 0 0" dist="${hand_length}"/>
   <!-- End effector -->
-  <link name="hand">
-    <xacro:prism_vci length="${hand_length}" side="${link_side}">
-      <origin xyz="0 0 ${hand_length/2}" rpy="0 0 0"/>
+  <link name="finger">
+    <xacro:prism_vci length="${finger_length}" side="${link_side}">
+      <origin xyz="0 0 ${finger_length/2}" rpy="0 0 0"/>
     </xacro:prism_vci>
   </link>
-  <gazebo reference="hand">
+  <gazebo reference="finger">
     <material>Gazebo/Red</material>
   </gazebo>

Commit message: last version

File: src/integ_description/urdf/arm.urdf.xacro (robot description, xacro)
@@ -1,20 +1,18 @@
 <?xml version="1.0"?>
 <robot name="arm" xmlns:xacro="http://www.ros.org/wiki/xacro">
+<!-- Geometrical properties -->
+  <xacro:arg name="mass1" default="1."/>
+  <xacro:arg name="mass2" default="0.5"/>
+  <xacro:arg name="hand_length" default="0.8"/>
+  <xacro:arg name="finger_length" default="0.6"/>
   <xacro:property name="PI" value="3.14159265359"/>
-  <!-- Joints Control in Gazebo -->
-  <gazebo>
-    <plugin name="gazebo_ros_control" filename="libgazebo_ros_control.so"/>
-  </gazebo>
-  <!-- Geometrical properties -->
   <xacro:property name="link_side" value="0.04"/>
   <xacro:property name="joint_radius" value="0.036"/>
   <xacro:property name="joint_length" value="0.05"/>
-  <xacro:property name="leg_length" value="0"/>
-  <xacro:property name="arm_length" value="0"/>
-  <xacro:property name="hand_length" value="0.8"/>
-  <xacro:property name="finger_length" value="0.6"/>
-  <xacro:property name="camera_link" value="0.05"/>
-  <xacro:property name="axel_offset" value="0.05"/>
-  <xacro:property name="height3" value="1"/>
+  <xacro:property name="arm_length" value="0.001"/>
+  <xacro:property name="finger_length" value="$(arg finger_length)"/>
+  <xacro:property name="mass1" value="$(arg mass1)"/>
+  <xacro:property name="mass2" value="$(arg mass2)"/>
+  <xacro:property name="hand_length" value="$(arg hand_length)"/>
   <!-- Materials -->
   <material name="orange">
@@ -24,9 +22,10 @@
     <color rgba="0.80 0.80 0.80 1.00"/>
   </material>
-  <material name="red">
-	  <color rgba="0.8 0.0 0.0 1.0"/>
-  </material
+  <!-- Joints Control in Gazebo -->
+  <gazebo>
+    <plugin name="gazebo_ros_control" filename="libgazebo_ros_control.so"/>
+  </gazebo>
   <!-- Generates a box visual/collision/inertial -->
-  <xacro:macro name="prism_vci" params="side length mass:=0.1 *origin">
+  <xacro:macro name="prism_vci" params="side length mass *origin">
     <xacro:macro name="prism_geometry">
       <xacro:insert_block name="origin"/>
@@ -48,24 +47,11 @@
     </inertial>
   </xacro:macro>
-  <!-- Generates a cylinder visual/collision -->
-  <xacro:macro name="cylinder_vc" params="radius length *origin">
-    <xacro:macro name="cylinder_geometry">
-      <xacro:insert_block name="origin"/>
-      <geometry>
-        <cylinder length="${length}" radius="${radius}"/>
-      </geometry>
-    </xacro:macro>
-    <visual>
-      <xacro:cylinder_geometry/>
-      <material name="gray"/>
-    </visual>
-  </xacro:macro>
   <!-- Generates child joint of parent -->
-  <xacro:macro name="arm_joint" params="child parent dist:=0 axis">
+  <xacro:macro name="arm_joint" params="child parent dist:=0 ">
     <joint name="${parent}_${child}_joint" type="revolute">
       <origin xyz="0 0 ${dist}" rpy="0 0 0"/>
       <parent link="${parent}"/>
       <child link="${child}"/>
-      <axis xyz="${axis}"/>
+      <axis xyz="1 0 0"/>
       <limit effort="40.0"
              velocity="1.0"
@@ -81,23 +67,18 @@
       <actuator name="${parent}_${child}_actuator"/>
     </transmission>
-    <link name="${parent}">
-      <xacro:prism_vci length="${dist}" side="${link_side}">
-        <origin xyz="0 0 ${dist/2}" rpy="0 0 0"/>
-      </xacro:prism_vci>
-      <xacro:cylinder_vc radius="${joint_radius}" length="${joint_length}">
-        <xacro:if value="${axis=='0 0 1'}">
-          <origin xyz="0 0 ${dist}" rpy="0 0 0"/>
-        </xacro:if>
-        <xacro:if value="${axis=='1 0 0'}">
-          <origin xyz="0 0 ${dist}" rpy="0 ${PI/2} 0"/>
-        </xacro:if>
-        <xacro:if value="${axis=='0 1 0'}">
-          <origin xyz="0 0 ${dist}" rpy="${PI/2} 0 0"/>
-        </xacro:if>
-      </xacro:cylinder_vc>
+  <!--Creating a visual for the joints-->
+    <joint name="${parent}_${child}_fixed" type="fixed">
+        <origin xyz="0 0 ${dist}" rpy="0 ${PI/2} 0"/>
+        <parent link="${parent}"/>
+        <child link="${child}_fixed"/>
+    </joint>
+    <link name="${child}_fixed">
+      <visual>
+        <geometry>
+          <cylinder length="${joint_length}" radius="${joint_radius}"/>
+        </geometry>
+        <material name="gray"/>
+      </visual>
     </link>
-    <gazebo reference="${parent}">
-      <material>Gazebo/Orange</material>
-    </gazebo>
   </xacro:macro>
   <!-- World frame (for Gazebo) -->
@@ -108,12 +89,29 @@
     <child link="arm"/>
   </joint>
-  <!--<xacro:arm_joint parent="world" child="arm" axis="0 0 1" dist="0"/>-->
   <!-- Joints Chain -->
-  <!--<xacro:arm_joint parent="leg" child="arm" axis="0 0 1" dist="${leg_length}"/>-->
-  <xacro:arm_joint parent="arm" child="hand" axis="1 0 0" dist="${arm_length}"/>
-  <xacro:arm_joint parent="hand" child="finger" axis="1 0 0" dist="${hand_length}"/>
+  <xacro:arm_joint parent="arm" child="hand" dist="${arm_length}"/>
+  <xacro:arm_joint parent="hand" child="finger" dist="$(arg hand_length)"/>
+ <!--LINKS-->
+ <!-- arm -->
+ <link name="arm">
+    <xacro:prism_vci length="${arm_length}" mass = "$(arg mass1)" side="${link_side}">
+      <origin xyz="0 0 ${arm_length/2}" rpy="0 0 0"/>
+    </xacro:prism_vci>
+  </link>
+  <gazebo reference="arm">
+    <material>Gazebo/Red</material>
+  </gazebo>
+ <!-- hand -->
+  <link name="hand">
+    <xacro:prism_vci length="${hand_length}" mass = "$(arg mass2)" side="${link_side}">
+      <origin xyz="0 0 ${hand_length/2}" rpy="0 0 0"/>
+    </xacro:prism_vci>
+  </link>
+  <gazebo reference="hand">
+    <material>Gazebo/Red</material>
+  </gazebo>
   <!-- End effector -->
   <link name="finger">
-    <xacro:prism_vci length="${finger_length}" side="${link_side}">
+    <xacro:prism_vci length="${finger_length}" mass = "$(arg mass2)" side="${link_side}">
       <origin xyz="0 0 ${finger_length/2}" rpy="0 0 0"/>
     </xacro:prism_vci>
@@ -122,70 +120,3 @@
     <material>Gazebo/Red</material>
   </gazebo>
-     <!-- Camera -->
-   <link name="camera_link">
-    <collision>
-      <origin xyz="0 0 0" rpy="0 0 0"/>
-      <geometry>
-    <box size="${camera_link} ${camera_link} ${camera_link}"/>
-      </geometry>
-    </collision>
-    <visual>
-      <origin xyz="0 0 0" rpy="0 0 0"/>
-      <geometry>
-    <box size="${camera_link} ${camera_link} ${camera_link}"/>
-      </geometry>
-      <material name="red"/>
-    </visual>
-    <inertial>
-      <mass value="1e-5" />
-      <origin xyz="0 0 0" rpy="0 0 0"/>
-      <inertia ixx="1e-6" ixy="0" ixz="0" iyy="1e-6" iyz="0" izz="1e-6" />
-    </inertial>
-  </link>
-   <joint name="camera_joint" type="fixed">
-    <axis xyz="0 1 0" />
-    <origin xyz="${camera_link} 0 ${height3 - axel_offset*2}" rpy="0 0 0"/>
-    <parent link="finger"/>
-    <child link="camera_link"/>
-  </joint>
-   <!-- camera -->
-  <gazebo reference="camera_link">
-    <sensor type="camera" name="camera1">
-      <update_rate>30.0</update_rate>
-      <camera name="head">
-        <horizontal_fov>1.3962634</horizontal_fov>
-        <image>
-          <width>800</width>
-          <height>800</height>
-          <format>R8G8B8</format>
-        </image>
-        <clip>
-          <near>0.02</near>
-          <far>300</far>
-        </clip>
-        <noise>
-          <type>gaussian</type>
-          <!-- Noise is sampled independently per pixel on each frame.
-               That pixel's noise value is added to each of its color
-               channels, which at that point lie in the range [0,1]. -->
-          <mean>0.0</mean>
-          <stddev>0.007</stddev>
-        </noise>
-      </camera>
-      <plugin name="camera_controller" filename="libgazebo_ros_camera.so">
-        <alwaysOn>true</alwaysOn>
-        <updateRate>0.0</updateRate>
-        <cameraName>robot/camera1</cameraName>
-        <imageTopicName>image_raw</imageTopicName>
-        <cameraInfoTopicName>camera_info</cameraInfoTopicName>
-        <frameName>camera_link</frameName>
-        <hackBaseline>0.07</hackBaseline>
-        <distortionK1>0.0</distortionK1>
-        <distortionK2>0.0</distortionK2>
-        <distortionK3>0.0</distortionK3>
-        <distortionT1>0.0</distortionT1>
-        <distortionT2>0.0</distortionT2>
-      </plugin>
-    </sensor>
-  </gazebo>
 </robot>

Commit message: Update arm.urdf.xacro

File: src/integ_description/urdf/arm.urdf.xacro (robot description, xacro)
@@ -120,3 +120,70 @@
     <material>Gazebo/Red</material>
   </gazebo>
+  <!-- Camera -->
+   <link name="camera_link">
+    <collision>
+      <origin xyz="0 0 0" rpy="0 0 0"/>
+      <geometry>
+    <box size="${camera_link} ${camera_link} ${camera_link}"/>
+      </geometry>
+    </collision>
+    <visual>
+      <origin xyz="0 0 0" rpy="0 0 0"/>
+      <geometry>
+    <box size="${camera_link} ${camera_link} ${camera_link}"/>
+      </geometry>
+      <material name="red"/>
+    </visual>
+    <inertial>
+      <mass value="1e-5" />
+      <origin xyz="0 0 0" rpy="0 0 0"/>
+      <inertia ixx="1e-6" ixy="0" ixz="0" iyy="1e-6" iyz="0" izz="1e-6" />
+    </inertial>
+  </link>
+   <joint name="camera_joint" type="fixed">
+    <axis xyz="0 1 0" />
+    <origin xyz="${camera_link} 0 ${height3 - axel_offset*2}" rpy="0 0 0"/>
+    <parent link="finger"/>
+    <child link="camera_link"/>
+  </joint>
+   <!-- camera -->
+  <gazebo reference="camera_link">
+    <sensor type="camera" name="camera1">
+      <update_rate>30.0</update_rate>
+      <camera name="head">
+        <horizontal_fov>1.3962634</horizontal_fov>
+        <image>
+          <width>800</width>
+          <height>800</height>
+          <format>R8G8B8</format>
+        </image>
+        <clip>
+          <near>0.02</near>
+          <far>300</far>
+        </clip>
+        <noise>
+          <type>gaussian</type>
+          <!-- Noise is sampled independently per pixel on each frame.
+               That pixel's noise value is added to each of its color
+               channels, which at that point lie in the range [0,1]. -->
+          <mean>0.0</mean>
+          <stddev>0.007</stddev>
+        </noise>
+      </camera>
+      <plugin name="camera_controller" filename="libgazebo_ros_camera.so">
+        <alwaysOn>true</alwaysOn>
+        <updateRate>0.0</updateRate>
+        <cameraName>robot/camera1</cameraName>
+        <imageTopicName>image_raw</imageTopicName>
+        <cameraInfoTopicName>camera_info</cameraInfoTopicName>
+        <frameName>camera_link</frameName>
+        <hackBaseline>0.07</hackBaseline>
+        <distortionK1>0.0</distortionK1>
+        <distortionK2>0.0</distortionK2>
+        <distortionK3>0.0</distortionK3>
+        <distortionT1>0.0</distortionT1>
+        <distortionT2>0.0</distortionT2>
+      </plugin>
+    </sensor>
+  </gazebo>
 </robot>

Commit message: Update arm.urdf.xacro

File: src/integ_description/urdf/arm.urdf.xacro (robot description, xacro)
@@ -15,4 +15,7 @@
   <xacro:property name="mass2" value="$(arg mass2)"/>
   <xacro:property name="hand_length" value="$(arg hand_length)"/>
+  <xacro:property name="camera_link" value="0.05"/>
+  <xacro:property name="axel_offset" value="0.05"/>
+  <xacro:property name="height3" value="1"/>
   <!-- Materials -->
   <material name="orange">
@@ -21,4 +24,7 @@
   <material name="gray">
     <color rgba="0.80 0.80 0.80 1.00"/>
+  </material>
+  <material name="red">
+	   <color rgba="0.8 0.0 0.0 1.0"/>
   </material>
   <!-- Joints Control in Gazebo -->

Commit message: disable strange camera_link references in xacro

File: src/integ_description/urdf/arm.urdf.xacro (robot description, xacro)
@@ -120,7 +120,7 @@
     <material>Gazebo/Red</material>
   </gazebo>
-  <!-- Camera -->
+  <!-- Camera not well defined-> go to 0, 0, 0 -->
    <link name="camera_link">
-    <collision>
+   <!-- <collision>
       <origin xyz="0 0 0" rpy="0 0 0"/>
       <geometry>
@@ -131,5 +131,5 @@
       <origin xyz="0 0 0" rpy="0 0 0"/>
       <geometry>
-    <box size="${camera_link} ${camera_link} ${camera_link}"/>
+        <box size="${camera_link} ${camera_link} ${camera_link}"/>
       </geometry>
       <material name="red"/>
@@ -139,9 +139,9 @@
       <origin xyz="0 0 0" rpy="0 0 0"/>
       <inertia ixx="1e-6" ixy="0" ixz="0" iyy="1e-6" iyz="0" izz="1e-6" />
-    </inertial>
+    </inertial>-->
   </link>
    <joint name="camera_joint" type="fixed">
     <axis xyz="0 1 0" />
-    <origin xyz="${camera_link} 0 ${height3 - axel_offset*2}" rpy="0 0 0"/>
+    <origin xyz="0 0 0" rpy="0 0 0"/>
     <parent link="finger"/>
     <child link="camera_link"/>

Commit message: with camera

File: src/integ_description/urdf/arm.urdf.xacro (robot description, xacro)
@@ -31,4 +31,5 @@
   <gazebo>
     <plugin name="gazebo_ros_control" filename="libgazebo_ros_control.so"/>
+    <robotNamespace>/</robotNamespace>
   </gazebo>
   <!-- Generates a box visual/collision/inertial -->
@@ -54,5 +55,5 @@
   </xacro:macro>
   <!-- Generates child joint of parent -->
-  <xacro:macro name="arm_joint" params="child parent dist:=0 ">
+  <xacro:macro name="arm_joint" params="child parent dist">
     <joint name="${parent}_${child}_joint" type="revolute">
       <origin xyz="0 0 ${dist}" rpy="0 0 0"/>
@@ -128,10 +129,4 @@
   <!-- Camera not well defined-> go to 0, 0, 0 -->
    <link name="camera_link">
-   <!-- <collision>
-      <origin xyz="0 0 0" rpy="0 0 0"/>
-      <geometry>
-    <box size="${camera_link} ${camera_link} ${camera_link}"/>
-      </geometry>
-    </collision>
     <visual>
       <origin xyz="0 0 0" rpy="0 0 0"/>
@@ -141,13 +136,7 @@
       <material name="red"/>
     </visual>
-    <inertial>
-      <mass value="1e-5" />
-      <origin xyz="0 0 0" rpy="0 0 0"/>
-      <inertia ixx="1e-6" ixy="0" ixz="0" iyy="1e-6" iyz="0" izz="1e-6" />
-    </inertial>-->
   </link>
    <joint name="camera_joint" type="fixed">
-    <axis xyz="0 1 0" />
-    <origin xyz="0 0 0" rpy="0 0 0"/>
+    <origin xyz="0 0 ${finger_length}" rpy="0 0 0"/>
     <parent link="finger"/>
     <child link="camera_link"/>

Commit message: camera axes consistent with computer vision

File: src/integ_description/urdf/arm.urdf.xacro (robot description, xacro)
@@ -61,6 +61,6 @@
       <child link="${child}"/>
       <axis xyz="1 0 0"/>
-      <limit effort="40.0"
-             velocity="1.0"
+      <limit effort="100.0"
+             velocity="10.0"
              lower="${-PI}"
              upper="${PI}"/>
@@ -138,5 +138,5 @@
   </link>
    <joint name="camera_joint" type="fixed">
-    <origin xyz="0 0 ${finger_length}" rpy="0 0 0"/>
+    <origin xyz="0 0 ${finger_length}" rpy="${-PI/2} 0 ${-PI/2}"/>
     <parent link="finger"/>
     <child link="camera_link"/>
@@ -147,4 +147,7 @@
       <update_rate>30.0</update_rate>
       <camera name="head">
+        <!-- Gazebo uses X as the optical axis -->
+          <visualize>true</visualize>
+          <pose>0 0 0 0 ${-PI/2} ${PI/2}</pose>
         <horizontal_fov>1.3962634</horizontal_fov>
         <image>
